File: 25kHz/FilterAndHalfBuffer/_autosave-FilterAndHalfBuffer.kicad_sch (KiCad schematic)
At the start: 36 parts, among them J1 IN_IN, J2 IN_QN, J3 PWR, J4 EXT_LED_PWR, J5 IN_IP, J7 IN_QP, J8 Conn_01x02, J9 Conn_01x02, U2 LM317_TO-220, U3 LM358

Commit message: Update PCB
Connections:
- net at R11.2, R14.2, U3.3 (+): no longer R12.1
- net at R13.1, U3.2 (-): now also R12.1
Changed lines of the file:
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@@
   (junction (at 58.42 45.72) (diameter 0) (color 0 0 0 0)
   )
-  (junction (at 72.39 40.64) (diameter 0) (color 0 0 0 0)
-  )
   (junction (at 65.405 141.605) (diameter 0) (color 0 0 0 0)
   )
@@
   (junction (at 130.81 153.67) (diameter 0) (color 0 0 0 0)
   )
+  (junction (at 72.39 45.72) (diameter 0) (color 0 0 0 0)
+  )
   (junction (at 163.83 34.925) (diameter 0) (color 0 0 0 0)
   )
@@
     (stroke (width 0) (type default))
   )
-  (wire (pts (xy 71.12 45.72) (xy 75.565 45.72))
-    (stroke (width 0) (type default))
-  )
   (wire (pts (xy 156.845 34.925) (xy 156.845 29.845))
     (stroke (width 0) (type default))
@@
     (stroke (width 0) (type default))
   )
-  (wire (pts (xy 72.39 40.64) (xy 73.66 40.64))
-    (stroke (width 0) (type default))
-  )
   (wire (pts (xy 71.12 83.185) (xy 73.025 83.185))
     (stroke (width 0) (type default))
@@
     (stroke (width 0) (type default))
   )
-  (wire (pts (xy 72.39 30.48) (xy 72.39 40.64))
-    (stroke (width 0) (type default))
-  )
   (wire (pts (xy 94.615 124.46) (xy 94.615 113.03))
     (stroke (width 0) (type default))
@@
     (stroke (width 0) (type default))
   )
-  (wire (pts (xy 71.12 40.64) (xy 72.39 40.64))
+  (wire (pts (xy 71.12 40.64) (xy 73.66 40.64))
     (stroke (width 0) (type default))
   )
@@
     (stroke (width 0) (type default))
   )
+  (wire (pts (xy 71.12 45.72) (xy 72.39 45.72))
+    (stroke (width 0) (type default))
+  )
   (wire (pts (xy 149.225 45.085) (xy 156.845 45.085))
     (stroke (width 0) (type default))
@@
     (stroke (width 0) (type default))
   )
+  (wire (pts (xy 72.39 45.72) (xy 75.565 45.72))
+    (stroke (width 0) (type default))
+  )
   (wire (pts (xy 156.845 29.845) (xy 149.225 29.845))
     (stroke (width 0) (type default))
@@
     (stroke (width 0) (type default))
   )
+  (wire (pts (xy 72.39 30.48) (xy 72.39 45.72))
+    (stroke (width 0) (type default))
+  )
